File: csi/csipmod/csipmod.sch (KiCad schematic (older format))
At the start: 38 parts

Commit message: csipmod: PCB ready to route
Signed-off-by: David Shah <davey1576@gmail.com>
Parts:
- C1, C3, C4: renamed from C?; footprint (none) -> Capacitor_SMD:C_0805_2012Metric
- C2: renamed from C?; footprint (none) -> Capacitor_SMD:C_0402_1005Metric
- J1, J2: renamed from J?; footprint (none) -> Custom Parts:PMOD_2x06_2.54mm
- P1: renamed from P?; footprint (none) -> Custom Parts:1-1734248-5
- R1, R10, R11, R12, R13, R14, R15, R16, R17, R18, R19, R2, R20, R21, R22, R23, R24, R25, R26, R27, R28, R3, R4, R5, R6, R7, R8, R9: renamed from R?; footprint (none) -> Resistor_SMD:R_0402_1005Metric
- R29: renamed from R?; footprint (none) -> Resistor_SMD:R_0805_2012Metric
- U2: renamed from U?; footprint (none) -> Package_SO:SSOP-8_2.95x2.8mm_P0.65mm
- gave numbers to parts that had none: 1
Connections:
- net labels added: CCLK+, CCLK-, CD0+, CD0-, CD1+, CD1-
